File: RocketBoardV2.kicad_sch (KiCad schematic)
At the start: 67 parts, among them IC1 W25Q256JVEIQ, J1 10118194-0001LF, J3 Conn_01x03_Pin, U1 SC0914_13_, U2 W25Q16JVUXIQ_TR, U3 BMI270, U4 TPS62420DRCR, Y1 ABM8-272-T3

Commit message: more finalized layout, placed C + R
Parts:
- C1, C10, C11, C12, C13, C14, C15, C16, C17, C18, C19, C2, C20, C21, C22, C23, C24, C25, C26, C3, C4, C5, C6, C7, C8, C9: footprint (none) -> Capacitor_SMD:C_0402_1005Metric
- D1, D2: footprint (none) -> LED_SMD:LED_0402_1005Metric
- L1, L2: footprint (none) -> Inductor_SMD:L_0402_1005Metric
- R1, R10, R11, R12, R13, R14, R15, R2, R3, R4, R5, R6, R7, R8, R9: footprint (none) -> Resistor_SMD:R_0402_1005Metric
- TP1, TP2: footprint (none) -> TestPoint:TestPoint_Pad_1.0x1.0mm
- U4: footprint TPS62420DRCR:IC_TPS62420DRCR -> Components:IC_TPS62420DRCR
Changed lines of the file:
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@@
 			)
 		)
-		(property "Footprint" ""
+		(property "Footprint" "Inductor_SMD:L_0402_1005Metric"
 			(at 490.22 113.03 0)
 			(effects
@@
 			)
 		)
-		(property "Footprint" ""
+		(property "Footprint" "Capacitor_SMD:C_0402_1005Metric"
 			(at 384.5052 232.41 0)
 			(effects
@@
 			)
 		)
-		(property "Footprint" ""
+		(property "Footprint" "Capacitor_SMD:C_0402_1005Metric"
 			(at 477.2152 121.92 0)
 			(effects
@@
 			)
 		)
-		(property "Footprint" ""
+		(property "Footprint" "Capacitor_SMD:C_0402_1005Metric"
 			(at 105.7148 234.95 0)
 			(effects
@@
 			)
 		)
-		(property "Footprint" ""
+		(property "Footprint" "Resistor_SMD:R_0402_1005Metric"
 			(at 104.902 217.17 90)
 			(effects
@@
 			)
 		)
-		(property "Footprint" ""
+		(property "Footprint" "Capacitor_SMD:C_0402_1005Metric"
 			(at 121.6152 332.74 0)
 			(effects
@@
 			)
 		)
-		(property "Footprint" "TPS62420DRCR:IC_TPS62420DRCR"
+		(property "Footprint" "Components:IC_TPS62420DRCR"
 			(at 514.35 100.33 0)
 			(effects
@@
 			)
 		)
-		(property "Footprint" ""
+		(property "Footprint" "Capacitor_SMD:C_0402_1005Metric"
 			(at 465.7852 121.92 0)
 			(effects
@@
 			)
 		)
-		(property "Footprint" ""
+		(property "Footprint" "Capacitor_SMD:C_0402_1005Metric"
 			(at 407.3652 232.41 0)
 			(effects
@@
 			)
 		)
-		(property "Footprint" ""
+		(property "Footprint" "LED_SMD:LED_0402_1005Metric"
 			(at 259.08 205.74 0)
 			(effects
@@
 			)
 		)
-		(property "Footprint" ""
+		(property "Footprint" "Capacitor_SMD:C_0402_1005Metric"
 			(at 376.8852 232.41 0)
 			(effects
@@
 			)
 		)
-		(property "Footprint" ""
+		(property "Footprint" "Capacitor_SMD:C_0402_1005Metric"
 			(at 225.7552 318.77 0)
 			(effects
@@
 			)
 		)
-		(property "Footprint" ""
+		(property "Footprint" "Capacitor_SMD:C_0402_1005Metric"
 			(at 414.9852 232.41 0)
 			(effects
@@
 			)
 		)
-		(property "Footprint" ""
+		(property "Footprint" "TestPoint:TestPoint_Pad_1.0x1.0mm"
 			(at 72.39 76.2 0)
 			(effects
@@
 			)
 		)
-		(property "Footprint" ""
+		(property "Footprint" "Capacitor_SMD:C_0402_1005Metric"
 			(at 234.6452 118.11 0)
 			(effects
@@
 			)
 		)
-		(property "Footprint" ""
+		(property "Footprint" "Resistor_SMD:R_0402_1005Metric"
 			(at 486.918 128.27 90)
 			(effects
@@
 			)
 		)
-		(property "Footprint" ""
+		(property "Footprint" "Capacitor_SMD:C_0402_1005Metric"
 			(at 381.3048 334.01 0)
 			(effects
@@
 			)
 		)
-		(property "Footprint" ""
+		(property "Footprint" "Capacitor_SMD:C_0402_1005Metric"
 			(at 263.1948 118.11 0)
 			(effects
@@
 			)
 		)
-		(property "Footprint" ""
+		(property "Footprint" "Resistor_SMD:R_0402_1005Metric"
 			(at 143.51 108.458 90)
 			(effects
@@
 			)
 		)
-		(property "Footprint" ""
+		(property "Footprint" "Capacitor_SMD:C_0402_1005Metric"
 			(at 58.7248 78.74 0)
 			(effects
@@
 			)
 		)
-		(property "Footprint" ""
+		(property "Footprint" "Capacitor_SMD:C_0402_1005Metric"
 			(at 491.1852 340.36 0)
 			(effects
@@
 			)
 		)
-		(property "Footprint" ""
+		(property "Footprint" "Resistor_SMD:R_0402_1005Metric"
 			(at 143.51 107.442 90)
 			(effects
@@
 			)
 		)
-		(property "Footprint" ""
+		(property "Footprint" "Capacitor_SMD:C_0402_1005Metric"
 			(at 378.1552 334.01 0)
 			(effects
@@
 			)
 		)
-		(property "Footprint" ""
+		(property "Footprint" "Resistor_SMD:R_0402_1005Metric"
 			(at 483.362 118.11 90)
 			(effects
@@
 			)
 		)
-		(property "Footprint" ""
+		(property "Footprint" "Capacitor_SMD:C_0402_1005Metric"
 			(at 216.2048 318.77 0)
 			(effects
@@
 			)
 		)
-		(property "Footprint" ""
+		(property "Footprint" "Capacitor_SMD:C_0402_1005Metric"
 			(at 166.6748 71.12 0)
 			(effects
@@
 			)
 		)
-		(property "Footprint" ""
+		(property "Footprint" "Resistor_SMD:R_0402_1005Metric"
 			(at 436.118 312.42 90)
 			(effects
@@
 			)
 		)
-		(property "Footprint" ""
+		(property "Footprint" "Capacitor_SMD:C_0402_1005Metric"
 			(at 399.7452 106.68 0)
 			(effects
@@
 			)
 		)
-		(property "Footprint" ""
+		(property "Footprint" "Capacitor_SMD:C_0402_1005Metric"
 			(at 174.9552 71.12 0)
 			(effects
@@
 			)
 		)
-		(property "Footprint" ""
+		(property "Footprint" "Capacitor_SMD:C_0402_1005Metric"
 			(at 472.1352 101.6 0)
 			(effects
@@
 			)
 		)
-		(property "Footprint" ""
+		(property "Footprint" "Capacitor_SMD:C_0402_1005Metric"
 			(at 392.1252 232.41 0)
 			(effects
@@
 			)
 		)
-		(property "Footprint" ""
+		(property "Footprint" "Resistor_SMD:R_0402_1005Metric"
 			(at 262.382 99.06 90)
 			(effects
@@
 			)
 		)
-		(property "Footprint" ""
+		(property "Footprint" "Capacitor_SMD:C_0402_1005Metric"
 			(at 399.7452 232.41 0)
 			(effects
@@
 			)
 		)
-		(property "Footprint" ""
+		(property "Footprint" "Capacitor_SMD:C_0402_1005Metric"
 			(at 494.3348 340.36 0)
 			(effects
@@
 			)
 		)
-		(property "Footprint" ""
+		(property "Footprint" "LED_SMD:LED_0402_1005Metric"
 			(at 259.08 224.79 0)
 			(effects
@@
 			)
 		)
-		(property "Footprint" ""
+		(property "Footprint" "Resistor_SMD:R_0402_1005Metric"
 			(at 314.198 312.42 90)
 			(effects
@@
 			)
 		)
-		(property "Footprint" ""
+		(property "Footprint" "Resistor_SMD:R_0402_1005Metric"
 			(at 247.65 207.518 90)
 			(effects
@@
 			)
 		)
-		(property "Footprint" ""
+		(property "Footprint" "Resistor_SMD:R_0402_1005Metric"
 			(at 485.648 97.79 90)
 			(effects
@@
 			)
 		)
-		(property "Footprint" ""
+		(property "Footprint" "Resistor_SMD:R_0402_1005Metric"
 			(at 494.538 312.42 90)
 			(effects
@@
 			)
 		)
-		(property "Footprint" ""
+		(property "Footprint" "Resistor_SMD:R_0402_1005Metric"
 			(at 319.532 312.42 90)
 			(effects
@@
 			)
 		)
-		(property "Footprint" ""
+		(property "Footprint" "Inductor_SMD:L_0402_1005Metric"
 			(at 490.22 92.71 0)
 			(effects
@@
 			)
 		)
-		(property "Footprint" ""
+		(property "Footprint" "Capacitor_SMD:C_0402_1005Metric"
 			(at 460.7052 93.98 0)
 			(effects
@@
 			)
 		)
-		(property "Footprint" ""
+		(property "Footprint" "Resistor_SMD:R_0402_1005Metric"
 			(at 477.52 101.092 90)
 			(effects
@@
 			)
 		)
-		(property "Footprint" ""
+		(property "Footprint" "Capacitor_SMD:C_0402_1005Metric"
 			(at 164.7952 93.98 0)
 			(effects
@@
 			)
 		)
-		(property "Footprint" ""
+		(property "Footprint" "Resistor_SMD:R_0402_1005Metric"
 			(at 247.65 226.568 90)
 			(effects
@@
 			)
 		)
-		(property "Footprint" ""
+		(property "Footprint" "Resistor_SMD:R_0402_1005Metric"
 			(at 440.182 312.42 90)
 			(effects
@@
 			)
 		)
-		(property "Footprint" ""
+		(property "Footprint" "Capacitor_SMD:C_0402_1005Metric"
 			(at 343.8652 106.68 0)
 			(effects
@@
 			)
 		)
-		(property "Footprint" ""
+		(property "Footprint" "TestPoint:TestPoint_Pad_1.0x1.0mm"
 			(at 67.31 76.2 0)
 			(effects

Commit message: starting to route
Parts:
- removed D3, D4: D, symbol Device:D
- removed S1, S2: TL3315NF250Q, Components:SW_TL3315NF250Q, symbol TL3315NF250Q:TL3315NF250Q
- added D5, D6: MSS1P4-M3_89A, Components:DIODE_MSS1P4-M3_89A, symbol MSS1P4-M3_89A:MSS1P4-M3_89A
- added LED1: WS2812B-MINI, easyeda2kicad:LED-SMD_4P-L3.5-W3.5-TL_WS2812B, symbol easyeda2kicad:WS2812B-MINI
- added SW1, SW2: TS-1077S-02026, easyeda2kicad:SW-SMD_L3.1-W3.1-P2.20-LS4.0, symbol easyeda2kicad:TS-1077S-02026
- D1: value GREEN -> BLUE
Connections:
- net +5V: now also D5.1, D6.1, LED1.1 (VDD)
- net BARO_CS: now also U1.3 (GPIO1); no longer U1.6 (GPIO4)
- net GND: now also LED1.3 (VSS), SW1.2, SW2.1
- net GYRO_CS: now also U1.6 (GPIO4); no longer U1.3 (GPIO1)
- net RUN: now also SW1.1
- net at C25.1, VR1.1 (OUTPUT): now also D6.2
- net USB-: now reaches R1.1, U1.46 (USB_DM)
- net at R10.1: now also SW2.2
- net RGB_LED: now reaches U1.36 (GPIO24)
- net RGB_LED: now also LED1.4 (DIN)
- net USB+: now reaches R2.1, U1.47 (USB_DP)
- net at J1.1 (VCC): now also D5.2
- no-connect marks 5 -> 30
Other:
- note added: "RGB LED"
- moved on the sheet: D1, D2, R13, R8
